File: hw/burrowlark-usb/boards/groundlark-field-head/02-controller-page-01.kicad_sch (KiCad schematic)
At the start: 9 parts, among them J2 SWD / 3V3 SENSE, J3 BOOT0 jumper, U1 STM32F042K6T6

Commit message: Implement Burrowlark B1 four-sensor magnetic array
Use four aligned RM3100 modules on a 30 mm grid with a common SPI trigger, independent data/DRDY lanes and preserved raw cohort timing. Add explicit calibrated averaging, quartet backpressure handling, firmware fault fixtures and the matching workbench/README model.

Keep physical USB, timing, cross-talk and noise qualification explicit. The full-suite DAQHAT assembly failures are reproduced on the unchanged baseline.
Parts:
- added R9: 100k, Groundlark:Resistor_SMD__R_0603_1608Metric, symbol Groundlark:Part_R9
Connections:
- net MAG_MISO0: now reaches U1.10 (PA4)
- net MAG_MISO1: now reaches U1.11 (PA5)
- net MAG_MISO2: now reaches U1.12 (PA6)
- net MAG_MISO3: now reaches U1.13 (PA7)
- net MAG_DRDY1: now reaches U1.15 (PB1)
- net MAG_DRDY2: now reaches U1.26 (PB3)
- net MAG_DRDY3: now reaches U1.27 (PB4)
- net MAG_SCK: now reaches U1.7 (PA1)
- net MAG_MOSI: now reaches U1.8 (PA2)
- net MAG_CSN: now reaches U1.9 (PA3)
- net MAG_CSN: now also R9.1
- net MAG_DRDY renamed MAG_DRDY0
- new net V3_SENSOR: R9.2
- no-connect marks 17 -> 7
Changed lines of the file:
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@@
-(kicad_sch (version 20230121) (generator eeschema) (paper "A3") (title_block (title "groundlark-field-head / 02-controller-page-01") (date "2026-09-23") (rev "A2 PROTOTYPE"))
+(kicad_sch (version 20230121) (generator eeschema) (paper "A3") (title_block (title "groundlark-field-head / 02-controller-page-01") (date "2026-10-12") (rev "B1 PROTOTYPE"))
 (symbol (lib_id "Groundlark:Part_U1") (at 45.72 57.150000000000006 0) (unit 1) (in_bom yes) (on_board yes) (dnp no)
               (property "Reference" "U1" (at 45.72 31.560000000000002 0) (effects (font (size 1.27 1.27))))
@@
 (wire (pts (xy 30.48 50.8) (xy 25.4 50.8)) (stroke (width 0) (type default)))
 (global_label "SENSOR_EN" (shape bidirectional) (at 25.4 50.8 180) (effects (font (size 0.9 0.9)) (justify right)))
-(no_connect (at 30.48 53.34))
-(no_connect (at 30.48 55.88))
-(no_connect (at 30.48 58.42))
-(no_connect (at 30.48 60.96))
-(no_connect (at 30.48 63.5))
-(no_connect (at 30.48 66.04))
-(no_connect (at 30.48 68.58))
+(wire (pts (xy 30.48 53.34) (xy 25.4 53.34)) (stroke (width 0) (type default)))
+(global_label "MAG_SCK" (shape bidirectional) (at 25.4 53.34 180) (effects (font (size 0.9 0.9)) (justify right)))
+(wire (pts (xy 30.48 55.88) (xy 25.4 55.88)) (stroke (width 0) (type default)))
+(global_label "MAG_MOSI" (shape bidirectional) (at 25.4 55.88 180) (effects (font (size 0.9 0.9)) (justify right)))
+(wire (pts (xy 30.48 58.42) (xy 25.4 58.42)) (stroke (width 0) (type default)))
+(global_label "MAG_CSN" (shape bidirectional) (at 25.4 58.42 180) (effects (font (size 0.9 0.9)) (justify right)))
+(wire (pts (xy 30.48 60.96) (xy 25.4 60.96)) (stroke (width 0) (type default)))
+(global_label "MAG_MISO0" (shape bidirectional) (at 25.4 60.96 180) (effects (font (size 0.9 0.9)) (justify right)))
+(wire (pts (xy 30.48 63.5) (xy 25.4 63.5)) (stroke (width 0) (type default)))
+(global_label "MAG_MISO1" (shape bidirectional) (at 25.4 63.5 180) (effects (font (size 0.9 0.9)) (justify right)))
+(wire (pts (xy 30.48 66.04) (xy 25.4 66.04)) (stroke (width 0) (type default)))
+(global_label "MAG_MISO2" (shape bidirectional) (at 25.4 66.04 180) (effects (font (size 0.9 0.9)) (justify right)))
+(wire (pts (xy 30.48 68.58) (xy 25.4 68.58)) (stroke (width 0) (type default)))
+(global_label "MAG_MISO3" (shape bidirectional) (at 25.4 68.58 180) (effects (font (size 0.9 0.9)) (justify right)))
 (wire (pts (xy 30.48 71.12) (xy 25.4 71.12)) (stroke (width 0) (type default)))
-(global_label "MAG_DRDY" (shape bidirectional) (at 25.4 71.12 180) (effects (font (size 0.9 0.9)) (justify right)))
-(no_connect (at 30.48 73.66))
+(global_label "MAG_DRDY0" (shape bidirectional) (at 25.4 71.12 180) (effects (font (size 0.9 0.9)) (justify right)))
+(wire (pts (xy 30.48 73.66) (xy 25.4 73.66)) (stroke (width 0) (type default)))
+(global_label "MAG_DRDY1" (shape bidirectional) (at 25.4 73.66 180) (effects (font (size 0.9 0.9)) (justify right)))
 (wire (pts (xy 30.48 76.2) (xy 25.4 76.2)) (stroke (width 0) (type default)))
 (global_label "GND" (shape bidirectional) (at 25.4 76.2 180) (effects (font (size 0.9 0.9)) (justify right)))
@@
 (global_label "SWCLK" (shape bidirectional) (at 66.04 55.88 0) (effects (font (size 0.9 0.9)) (justify left)))
 (no_connect (at 60.96 58.42))
-(no_connect (at 60.96 60.96))
-(no_connect (at 60.96 63.5))
+(wire (pts (xy 60.96 60.96) (xy 66.04 60.96)) (stroke (width 0) (type default)))
+(global_label "MAG_DRDY2" (shape bidirectional) (at 66.04 60.96 0) (effects (font (size 0.9 0.9)) (justify left)))
+(wire (pts (xy 60.96 63.5) (xy 66.04 63.5)) (stroke (width 0) (type default)))
+(global_label "MAG_DRDY3" (shape bidirectional) (at 66.04 63.5 0) (effects (font (size 0.9 0.9)) (justify left)))
 (no_connect (at 60.96 66.04))
 (wire (pts (xy 60.96 68.58) (xy 66.04 68.58)) (stroke (width 0) (type default)))
@@
 (wire (pts (xy 60.96 137.16) (xy 66.04 137.16)) (stroke (width 0) (type default)))
 (global_label "BOOT0" (shape bidirectional) (at 66.04 137.16 0) (effects (font (size 0.9 0.9)) (justify left)))
+(symbol (lib_id "Groundlark:Part_R9") (at 142.24 137.16 0) (unit 1) (in_bom yes) (on_board yes) (dnp no)
+              (property "Reference" "R9" (at 142.24 130.62 0) (effects (font (size 1.27 1.27))))
+              (property "Value" "100k" (at 142.24 133.12 0) (effects (font (size 1.0 1.0))))
+              (property "Footprint" "Groundlark:Resistor_SMD__R_0603_1608Metric" (at 142.24 137.16 0) (effects (font (size 1 1)) hide))
+              (property "MPN" "RC0603FR-07100KL" (at 142.24 137.16 0) (effects (font (size 1 1)) hide))
+              (instances (project "groundlark-field-head" (path "/e1043b90-5a3a-5d7b-9b91-8488ec3f38a4/fc7d5532-6c14-5c58-945d-ed7a9463f825" (reference "R9") (unit 1)))))
+(wire (pts (xy 127.0 137.16) (xy 121.92 137.16)) (stroke (width 0) (type default)))
+(global_label "MAG_CSN" (shape bidirectional) (at 121.92 137.16 180) (effects (font (size 0.9 0.9)) (justify right)))
+(wire (pts (xy 157.48 137.16) (xy 162.56 137.16)) (stroke (width 0) (type default)))
+(global_label "V3_SENSOR" (shape bidirectional) (at 162.56 137.16 0) (effects (font (size 0.9 0.9)) (justify left)))
 )
