File: hw/burrowlark-usb/boards/groundlark-field-head/03-sensors-page-01.kicad_sch (KiCad schematic)
At the start: 9 parts, among them U2 RM3100 XYZ, U5 TPS22919, U6 SHT45

Commit message: Implement Burrowlark B1 four-sensor magnetic array
Use four aligned RM3100 modules on a 30 mm grid with a common SPI trigger, independent data/DRDY lanes and preserved raw cohort timing. Add explicit calibrated averaging, quartet backpressure handling, firmware fault fixtures and the matching workbench/README model.

Keep physical USB, timing, cross-talk and noise qualification explicit. The full-suite DAQHAT assembly failures are reproduced on the unchanged baseline.
Parts:
- removed C4: 100n, Groundlark:Capacitor_SMD__C_0603_1608Metric, symbol Groundlark:Part_C4
- removed U2: RM3100 XYZ, Groundlark:Groundlark__PNI_14190_Module, symbol Groundlark:Part_U2
Connections:
- no-connect marks 5 -> 1
Other:
- moved on the sheet: C10, U6
Changed lines of the file:
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@@
-(kicad_sch (version 20230121) (generator eeschema) (paper "A3") (title_block (title "groundlark-field-head / 03-sensors-page-01") (date "2026-09-23") (rev "A2 PROTOTYPE"))
+(kicad_sch (version 20230121) (generator eeschema) (paper "A3") (title_block (title "groundlark-field-head / 03-sensors-page-01") (date "2026-10-12") (rev "B1 PROTOTYPE"))
 (symbol (lib_id "Groundlark:Part_U5") (at 45.72 40.64 0) (unit 1) (in_bom yes) (on_board yes) (dnp no)
               (property "Reference" "U5" (at 45.72 31.560000000000002 0) (effects (font (size 1.27 1.27))))
@@
 (wire (pts (xy 60.96 71.12) (xy 66.04 71.12)) (stroke (width 0) (type default)))
 (global_label "V3_SENSOR" (shape bidirectional) (at 66.04 71.12 0) (effects (font (size 0.9 0.9)) (justify left)))
-(symbol (lib_id "Groundlark:Part_U2") (at 142.24 78.74 0) (unit 1) (in_bom yes) (on_board yes) (dnp no)
-              (property "Reference" "U2" (at 142.24 64.58 0) (effects (font (size 1.27 1.27))))
-              (property "Value" "RM3100 XYZ" (at 142.24 67.08 0) (effects (font (size 1.0 1.0))))
-              (property "Footprint" "Groundlark:Groundlark__PNI_14190_Module" (at 142.24 78.74 0) (effects (font (size 1 1)) hide))
-              (property "MPN" "PNI 14190" (at 142.24 78.74 0) (effects (font (size 1 1)) hide))
-              (instances (project "groundlark-field-head" (path "/e1043b90-5a3a-5d7b-9b91-8488ec3f38a4/ab979e54-c171-5922-9bbc-4aaabc504545" (reference "U2") (unit 1)))))
+(symbol (lib_id "Groundlark:Part_U6") (at 142.24 72.39 0) (unit 1) (in_bom yes) (on_board yes) (dnp no)
+              (property "Reference" "U6" (at 142.24 64.58 0) (effects (font (size 1.27 1.27))))
+              (property "Value" "SHT45" (at 142.24 67.08 0) (effects (font (size 1.0 1.0))))
+              (property "Footprint" "Groundlark:SHT45" (at 142.24 72.39 0) (effects (font (size 1 1)) hide))
+              (property "MPN" "SHT45-AD1B-R2" (at 142.24 72.39 0) (effects (font (size 1 1)) hide))
+              (instances (project "groundlark-field-head" (path "/e1043b90-5a3a-5d7b-9b91-8488ec3f38a4/ab979e54-c171-5922-9bbc-4aaabc504545" (reference "U6") (unit 1)))))
 (wire (pts (xy 127.0 71.12) (xy 121.92 71.12)) (stroke (width 0) (type default)))
-(global_label "SCL" (shape bidirectional) (at 121.92 71.12 180) (effects (font (size 0.9 0.9)) (justify right)))
+(global_label "SDA" (shape bidirectional) (at 121.92 71.12 180) (effects (font (size 0.9 0.9)) (justify right)))
 (wire (pts (xy 127.0 73.66) (xy 121.92 73.66)) (stroke (width 0) (type default)))
-(global_label "GND" (shape bidirectional) (at 121.92 73.66 180) (effects (font (size 0.9 0.9)) (justify right)))
-(wire (pts (xy 127.0 76.2) (xy 121.92 76.2)) (stroke (width 0) (type default)))
-(global_label "SDA" (shape bidirectional) (at 121.92 76.2 180) (effects (font (size 0.9 0.9)) (justify right)))
-(wire (pts (xy 127.0 78.74) (xy 121.92 78.74)) (stroke (width 0) (type default)))
-(global_label "GND" (shape bidirectional) (at 121.92 78.74 180) (effects (font (size 0.9 0.9)) (justify right)))
-(wire (pts (xy 127.0 81.28) (xy 121.92 81.28)) (stroke (width 0) (type default)))
-(global_label "MAG_DRDY" (shape bidirectional) (at 121.92 81.28 180) (effects (font (size 0.9 0.9)) (justify right)))
-(no_connect (at 127.0 83.82))
-(wire (pts (xy 127.0 86.36) (xy 121.92 86.36)) (stroke (width 0) (type default)))
-(global_label "GND" (shape bidirectional) (at 121.92 86.36 180) (effects (font (size 0.9 0.9)) (justify right)))
-(no_connect (at 157.48 71.12))
-(no_connect (at 157.48 73.66))
-(wire (pts (xy 157.48 76.2) (xy 162.56 76.2)) (stroke (width 0) (type default)))
-(global_label "V3_SENSOR" (shape bidirectional) (at 162.56 76.2 0) (effects (font (size 0.9 0.9)) (justify left)))
-(no_connect (at 157.48 78.74))
-(wire (pts (xy 157.48 81.28) (xy 162.56 81.28)) (stroke (width 0) (type default)))
-(global_label "V3_SENSOR" (shape bidirectional) (at 162.56 81.28 0) (effects (font (size 0.9 0.9)) (justify left)))
-(wire (pts (xy 157.48 83.82) (xy 162.56 83.82)) (stroke (width 0) (type default)))
-(global_label "V3_SENSOR" (shape bidirectional) (at 162.56 83.82 0) (effects (font (size 0.9 0.9)) (justify left)))
-(wire (pts (xy 157.48 86.36) (xy 162.56 86.36)) (stroke (width 0) (type default)))
-(global_label "GND" (shape bidirectional) (at 162.56 86.36 0) (effects (font (size 0.9 0.9)) (justify left)))
-(symbol (lib_id "Groundlark:Part_C4") (at 238.76 71.12 0) (unit 1) (in_bom yes) (on_board yes) (dnp no)
-              (property "Reference" "C4" (at 238.76 64.58 0) (effects (font (size 1.27 1.27))))
+(global_label "SCL" (shape bidirectional) (at 121.92 73.66 180) (effects (font (size 0.9 0.9)) (justify right)))
+(wire (pts (xy 157.48 71.12) (xy 162.56 71.12)) (stroke (width 0) (type default)))
+(global_label "V3_SENSOR" (shape bidirectional) (at 162.56 71.12 0) (effects (font (size 0.9 0.9)) (justify left)))
+(wire (pts (xy 157.48 73.66) (xy 162.56 73.66)) (stroke (width 0) (type default)))
+(global_label "GND" (shape bidirectional) (at 162.56 73.66 0) (effects (font (size 0.9 0.9)) (justify left)))
+(symbol (lib_id "Groundlark:Part_C10") (at 238.76 71.12 0) (unit 1) (in_bom yes) (on_board yes) (dnp no)
+              (property "Reference" "C10" (at 238.76 64.58 0) (effects (font (size 1.27 1.27))))
               (property "Value" "100n" (at 238.76 67.08 0) (effects (font (size 1.0 1.0))))
               (property "Footprint" "Groundlark:Capacitor_SMD__C_0603_1608Metric" (at 238.76 71.12 0) (effects (font (size 1 1)) hide))
               (property "MPN" "GRM188R71H104KA93D" (at 238.76 71.12 0) (effects (font (size 1 1)) hide))
-              (instances (project "groundlark-field-head" (path "/e1043b90-5a3a-5d7b-9b91-8488ec3f38a4/ab979e54-c171-5922-9bbc-4aaabc504545" (reference "C4") (unit 1)))))
+              (instances (project "groundlark-field-head" (path "/e1043b90-5a3a-5d7b-9b91-8488ec3f38a4/ab979e54-c171-5922-9bbc-4aaabc504545" (reference "C10") (unit 1)))))
 (wire (pts (xy 223.52 71.12) (xy 218.44 71.12)) (stroke (width 0) (type default)))
 (global_label "V3_SENSOR" (shape bidirectional) (at 218.44 71.12 180) (effects (font (size 0.9 0.9)) (justify right)))
 (wire (pts (xy 254.0 71.12) (xy 259.08 71.12)) (stroke (width 0) (type default)))
 (global_label "GND" (shape bidirectional) (at 259.08 71.12 0) (effects (font (size 0.9 0.9)) (justify left)))
-(symbol (lib_id "Groundlark:Part_U6") (at 335.28 72.39 0) (unit 1) (in_bom yes) (on_board yes) (dnp no)
-              (property "Reference" "U6" (at 335.28 64.58 0) (effects (font (size 1.27 1.27))))
-              (property "Value" "SHT45" (at 335.28 67.08 0) (effects (font (size 1.0 1.0))))
-              (property "Footprint" "Groundlark:SHT45" (at 335.28 72.39 0) (effects (font (size 1 1)) hide))
-              (property "MPN" "SHT45-AD1B-R2" (at 335.28 72.39 0) (effects (font (size 1 1)) hide))
-              (instances (project "groundlark-field-head" (path "/e1043b90-5a3a-5d7b-9b91-8488ec3f38a4/ab979e54-c171-5922-9bbc-4aaabc504545" (reference "U6") (unit 1)))))
-(wire (pts (xy 320.04 71.12) (xy 314.96 71.12)) (stroke (width 0) (type default)))
-(global_label "SDA" (shape bidirectional) (at 314.96 71.12 180) (effects (font (size 0.9 0.9)) (justify right)))
-(wire (pts (xy 320.04 73.66) (xy 314.96 73.66)) (stroke (width 0) (type default)))
-(global_label "SCL" (shape bidirectional) (at 314.96 73.66 180) (effects (font (size 0.9 0.9)) (justify right)))
-(wire (pts (xy 350.52 71.12) (xy 355.6 71.12)) (stroke (width 0) (type default)))
-(global_label "V3_SENSOR" (shape bidirectional) (at 355.6 71.12 0) (effects (font (size 0.9 0.9)) (justify left)))
-(wire (pts (xy 350.52 73.66) (xy 355.6 73.66)) (stroke (width 0) (type default)))
-(global_label "GND" (shape bidirectional) (at 355.6 73.66 0) (effects (font (size 0.9 0.9)) (justify left)))
-(symbol (lib_id "Groundlark:Part_C10") (at 45.72 114.3 0) (unit 1) (in_bom yes) (on_board yes) (dnp no)
-              (property "Reference" "C10" (at 45.72 107.75999999999999 0) (effects (font (size 1.27 1.27))))
-              (property "Value" "100n" (at 45.72 110.25999999999999 0) (effects (font (size 1.0 1.0))))
-              (property "Footprint" "Groundlark:Capacitor_SMD__C_0603_1608Metric" (at 45.72 114.3 0) (effects (font (size 1 1)) hide))
-              (property "MPN" "GRM188R71H104KA93D" (at 45.72 114.3 0) (effects (font (size 1 1)) hide))
-              (instances (project "groundlark-field-head" (path "/e1043b90-5a3a-5d7b-9b91-8488ec3f38a4/ab979e54-c171-5922-9bbc-4aaabc504545" (reference "C10") (unit 1)))))
-(wire (pts (xy 30.48 114.3) (xy 25.4 114.3)) (stroke (width 0) (type default)))
-(global_label "V3_SENSOR" (shape bidirectional) (at 25.4 114.3 180) (effects (font (size 0.9 0.9)) (justify right)))
-(wire (pts (xy 60.96 114.3) (xy 66.04 114.3)) (stroke (width 0) (type default)))
-(global_label "GND" (shape bidirectional) (at 66.04 114.3 0) (effects (font (size 0.9 0.9)) (justify left)))
 )
