File: hw/burrowlark-usb/layout/field_head/field_head.kicad_pcb (KiCad board)
At the start: 2 copper layers, 27 parts

Commit message: Implement Burrowlark B1 four-sensor magnetic array
Use four aligned RM3100 modules on a 30 mm grid with a common SPI trigger, independent data/DRDY lanes and preserved raw cohort timing. Add explicit calibrated averaging, quartet backpressure handling, firmware fault fixtures and the matching workbench/README model.

Keep physical USB, timing, cross-talk and noise qualification explicit. The full-suite DAQHAT assembly failures are reproduced on the unchanged baseline.
Parts:
- added C11: , elec:Capacitor_SMD__C_0603_1608Metric, F.Cu at (10.0, 0.00)
- added C12: , elec:Capacitor_SMD__C_0603_1608Metric, F.Cu at (30.0, 0.00)
- added C13: , elec:Capacitor_SMD__C_0603_1608Metric, F.Cu at (50.0, 0.00)
- added R9: , elec:Resistor_SMD__R_0603_1608Metric, F.Cu at (60.0, 0.00)
- added U7: , elec:Groundlark__PNI_14190_Module, F.Cu at (0.00, 0.00)
- added U8: , elec:Groundlark__PNI_14190_Module, F.Cu at (20.0, 0.00)
- added U9: , elec:Groundlark__PNI_14190_Module, F.Cu at (40.0, 0.00)
Connections:
- net MAG_DRDY renamed MAG_DRDY0
- U1 pad 10: 10 -> MAG_MISO0
- U1 pad 11: 11 -> MAG_MISO1
- U1 pad 12: 12 -> MAG_MISO2
- U1 pad 13: 13 -> MAG_MISO3
- U1 pad 15: 15 -> MAG_DRDY1
- U1 pad 26: 26 -> MAG_DRDY2
- U1 pad 27: 27 -> MAG_DRDY3
- U1 pad 7: 7 -> MAG_SCK
- U1 pad 8: 8 -> MAG_MOSI
- U1 pad 9: 9 -> MAG_CSN
- U2 pad 1: SCL -> MAG_SCK
- U2 pad 10: V3_SENSOR -> GND
- U2 pad 11: u2-11 -> 11
- U2 pad 2: GND -> MAG_MISO0
- U2 pad 3: SDA -> MAG_MOSI
- U2 pad 4: GND -> MAG_CSN
- U2 pad 8: u2-8 -> 8
- U2 pad 9: u2-9 -> 9
