File: hw/groundlark-fpga-hat/boards/groundlark-daqhat-01/03-geophone-page-01.kicad_sch (KiCad schematic)
At the start: 12 parts, among them J90 GEO + / - / SHIELD, U22 ADS122C04

Commit message: Update DAQHAT pressure sensor and assembly sourcing
Replace D90 with TPD2E2U06QDCKRQ1 and redesign U23 around SDP32-125PA. Synchronize routed CAD, native SES, models, supplier records, acquisition drivers, contracts, simulations, tests and documentation.

Record dated stock checks for 71 catalog identities and preserve the release gate for 52 unverified supplier placements. Generated manufacturing packages remain local and ignored.

Validation: repository structure and diff checks pass; prior full lab run passed 25 of 26 stages, with 301 software tests and 221 of 222 hardware tests passing. The remaining hardware test blocks unverified placements. Browser interaction and physical qualification remain pending.
Parts:
- D90: MPN TPD2E2U06DCKR -> TPD2E2U06QDCKRQ1
Changed lines of the file:
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@@
               (property "Value" "TPD2E2U06" (at 243.83999999999997 34.06 0) (effects (font (size 1.0 1.0))))
               (property "Footprint" "Groundlark:Package_TO_SOT_SMD__SOT-323_SC-70" (at 243.83999999999997 39.370000000000005 0) (effects (font (size 1 1)) hide))
-              (property "MPN" "TPD2E2U06DCKR" (at 243.83999999999997 39.370000000000005 0) (effects (font (size 1 1)) hide))
+              (property "MPN" "TPD2E2U06QDCKRQ1" (at 243.83999999999997 39.370000000000005 0) (effects (font (size 1 1)) hide))
               (instances (project "groundlark-daqhat-01" (path "/de5c43d7-546f-5b4d-b587-d8dfceb38170/fc4af920-ec4d-5175-b830-5c947dce5acb" (reference "D90") (unit 1)))))
 (wire (pts (xy 228.6 38.1) (xy 223.52 38.1)) (stroke (width 0) (type default)))
