File: hw/groundlark-fpga-hat/boards/groundlark-daqhat-01/groundlark-daqhat-01.kicad_sch (KiCad schematic)
At the start: 0 parts

Commit message: Strengthen DAQHAT power copper and validate native layout
Extend Pi supply pours to J1, add output via arrays and an FPGA distribution
bridge, spread D130 heat, correct GNSS RF width, and add UART idle bias.
Synchronize circuit, native CAD, schematic, SES, models and assembly mapping.

Extract native DC resistance, screen adjacent-layer coupling, preserve checks
under Python optimization, and disable I2C/I3C on the shared SPI IMUs.
Refresh specifications, supplier identity records and validation evidence.

Native ERC/DRC, route replay, simulations and 302 software tests pass. The final
hardware run passes 234/235; 52 supplier placement holds still prevent release.
All 71 exact catalog identities passed a fresh public inventory check.
Other:
- added sheet 07-fpga-host-isolation-page-02 (07-fpga-host-isolation-page-02.kicad_sch)
