File: hw/groundlark-fpga-hat/boards/groundlark-daqhat-01/04-gnss-page-01.kicad_sch (KiCad schematic)
At the start: 12 parts, among them J140 GNSS ANT / 3V3, U140 TPS70933, U141 TPS2553, U21 MAX-M10S-00B

Commit message: Fix GNSS RF margin and broaden pressure filter robustness
Parts:
- L140: value 27n -> 56n; footprint Groundlark:GNSS_L0402 -> Groundlark:GNSS_HP0402; MPN LQW15AN27NJ00D -> 0402HPH-56NXJRW
Connections:
- net GNSS_RF: no longer C148.2
- new net GNSS_MATCH: C148.2
Changed lines of the file:
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@@
 (global_label "GNSS_ANT" (shape bidirectional) (at 30.48 86.36 180) (effects (font (size 0.9 0.9)) (justify right)))
 (wire (pts (xy 66.04 86.36) (xy 71.12 86.36)) (stroke (width 0) (type default)))
-(global_label "GNSS_RF" (shape bidirectional) (at 71.12 86.36 0) (effects (font (size 0.9 0.9)) (justify left)))
+(global_label "GNSS_MATCH" (shape bidirectional) (at 71.12 86.36 0) (effects (font (size 0.9 0.9)) (justify left)))
 (symbol (lib_id "Groundlark:Part_L140") (at 147.32 86.36 0) (unit 1) (in_bom yes) (on_board yes) (dnp no)
               (property "Reference" "L140" (at 147.32 79.82 0) (effects (font (size 1.27 1.27))))
-              (property "Value" "27n" (at 147.32 82.32 0) (effects (font (size 1.0 1.0))))
-              (property "Footprint" "Groundlark:GNSS_L0402" (at 147.32 86.36 0) (effects (font (size 1 1)) hide))
-              (property "MPN" "LQW15AN27NJ00D" (at 147.32 86.36 0) (effects (font (size 1 1)) hide))
+              (property "Value" "56n" (at 147.32 82.32 0) (effects (font (size 1.0 1.0))))
+              (property "Footprint" "Groundlark:GNSS_HP0402" (at 147.32 86.36 0) (effects (font (size 1 1)) hide))
+              (property "MPN" "0402HPH-56NXJRW" (at 147.32 86.36 0) (effects (font (size 1 1)) hide))
               (instances (project "groundlark-daqhat-01" (path "/de5c43d7-546f-5b4d-b587-d8dfceb38170/63456fc1-bcd1-564c-918b-1145ac1e9ff5" (reference "L140") (unit 1)))))
 (wire (pts (xy 132.08 86.36) (xy 127.0 86.36)) (stroke (width 0) (type default)))
