File: hw/groundlark-fpga-hat/boards/groundlark-daqhat-01/stack-service-envelopes.kicad_pcb (KiCad board)
At the start: 6 copper layers, 140 x 56 mm, 208 parts, among them J1 Raspberry Pi 40-pin, J130 PI BATTERY 8-18V, J131 SWD / 3V3 REF, J140 GNSS ANT / 3V3, J4 FPGA test UART/reset, J80 LSHM-150-04.0-L-DV-A-S-K-TR, J81 LSHM-150-04.0-L-DV-A-S-K-TR, J82 LSHM-130-04.0-L-DV-A-S-K-TR, J83 12V DC / CENTER +, J90 GEO + / - / SHIELD, Q1 2N7002, Q130 2N7002, Q131 2N7002, SW80 FPGA OFF / ON, U1 24LC32A, U100 TMUX1574PWR, U101 TMUX1574PWR, U102 TCA9534PWR, U103 SN74LVC1G10DCKR, U104 TLV809EA30DBZR, U105 TLV809EA30DBZR, U106 SN74LVC1G08DCKR, U11 LSM6DSOTR, U12 LSM6DSOTR, U13 LSM6DSOTR, U130 MSPM0L1106, U131 TPS70933, U132 TPSM53603, U133 TPS22953, U140 TPS70933, U141 TPS2553, U21 MAX-M10S-00B, U22 ADS122C04, U23 SDP32-125PA, U40 TLV1117LV33DCYR, U41 SN74LVC8T245PWR, U42 SN74LVC8T245PWR, U43 ISO1640BDR, U51 TXU0202DCUR, U52 TLV803EA30DBZR, U80 TPSM53603

Commit message: Fix GNSS RF margin and broaden pressure filter robustness
Parts:
- added L141: 3.6n, Groundlark:GNSS_HP0402, B.Cu at (57.0, 65.8)
- C151, D140: moved to B.Cu
- L140: value 27n -> 56n; footprint Groundlark:GNSS_L0402 -> Groundlark:GNSS_HP0402; moved to B.Cu
- moved D140 4.00 mm to (54.0, 67.2)
- moved C151 3.07 mm to (55.0, 61.7)
- moved L140 2.80 mm to (54.0, 64.3)
- moved C148 1.27 mm to (55.5, 64.9)
Connections:
- C148 pad 2: GNSS_RF -> GNSS_MATCH
Routing:
- net GNSS_ANT: track 10.5 -> 3.18 mm
- net GND: track 687.1 -> 682.5 mm, vias 151 -> 153
- net GNSS_BIAS: track 10.0 -> 14.6 mm, vias 0 -> 1
- net GNSS_MATCH: track 0.00 -> 1.06 mm

Commit message: Resolve adjacent-layer coupling gate with revised signal routing
Routing:
- net IMU3_INT: track 57.6 -> 62.0 mm
- net PI_IMU3_CS: track 30.8 -> 34.6 mm
- net ID_SDA: track 46.7 -> 50.1 mm
- net LINK_DQ2: track 42.8 -> 46.2 mm, vias 7 -> 6
- net IMU3_CS: track 68.2 -> 70.9 mm
- net PI_IMU1_INT: track 78.2 -> 75.7 mm
- net I2C_SCL: track 85.9 -> 84.2 mm
- net PI_SPI_MISO: track 43.0 -> 44.7 mm
- net EEP_WP: track 78.8 -> 80.3 mm
- net PI_IMU1_CS: track 44.0 -> 45.3 mm
- net PI_IMU2_CS: track 37.9 -> 39.1 mm
- net PI_SPI_SCLK: track 40.7 -> 41.9 mm
- net ID_SCL: track 48.7 -> 49.5 mm
- net LINK_JTAG_SEL: track 56.4 -> 57.2 mm
- net FPGA_RESET_GPIO: track 56.3 -> 55.5 mm
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